File: pcb/krampus.sch (KiCad schematic (older format))
At the start: 2 parts

Commit message: power and pwm
Connections:
- net LSERVO: now reaches U?.10 (TC0W01/SERCOM0P1/Y3/AIN1/AIN5/PA05)
- net RSERVO: now reaches U?.11 (TC1WO0/SERCOM0P2/Y4/AIN2/AIN6/PA06)
Changed lines of the file:
@@
 	4000 1300 3650 1300
 Connection ~ 3650 1300
+Text GLabel 5950 2200 2    39   Input ~ 0
+LSERVO
+Text GLabel 5950 2300 2    39   Input ~ 0
+RSERVO
+Wire Wire Line
+	5600 2300 5950 2300
+Wire Wire Line
+	5600 2200 5950 2200
 $EndSCHEMATC
